Commit message: Fix sim hexapod gait: body_clearance 0.154→0.135, foot z -0.158→-0.140, foot_x 0.12→0.085
The default foot pose (0.12, 0, -0.158) sat 12mm OUTSIDE the leg's reach
(FEMUR+TIBIA=0.164). Every ik_coxa() call returned (0,0,0), which collapses
the leg horizontally, removes vertical support, and lets the body pancake
onto the floor. The sim then 'moves' but the legs sweep horizontally — the
robot drags itself rather than walking.

Changes:
- spooder.xacro base_joint z lowered from 0.154 to 0.135 (19mm lower body).
- nominal_stance_height lowered from -0.158 to -0.140 (foot 5mm below floor
  for stable single-point contact).
- nominal_stance_forward reduced from 0.12 to 0.085 — gives ~18mm reach
  margin at default and ~4cm forward step (AEP up to x=0.128).
- kinematics.ik_coxa() now clamps unreachable targets via clamp_to_reach()
  instead of silently returning (0,0,0); the gait can't collapse on bad IK.
- kinematics.clamp_to_reach() also pulls z toward 0 when |z| > FEMUR+TIBIA,
  so extreme targets don't bypass the leg-length limit.
- foothold_planner_node.py default + comment updated to the new stance.
- spooder_control/gait_controller.py BASE_FOOTPRINT_TO_BASE_LINK_Z drops
  from 0.154 to 0.135 to match.
- start_no_lidar.sh spawn_z lowered from 1.0 to 0.30 to reduce pancake
  risk during the bringup delay (gait controller starts ~16s post-spawn).
- test_navigation::test_kinematics assertions updated to expect the new
  clamping behavior instead of (0,0,0).

Verified reachable at (0.085, 0, -0.140): femur-tibia distance = 0.146,
~18mm inside the 0.164 outer reach. Forward stride ≈ 4cm/rear ≈ 12cm.
Predicted walking speed at vx=0.1 m/s, swing_dur=0.5s: ~0.05 m/s avg.

File: src/spooder_description/urdf/spooder.xacro (robot description, xacro)
@@ -9,7 +9,7 @@
   <xacro:property name="femur_length" value="0.060"/>
   <xacro:property name="tibia_length" value="0.104"/>
-  <!-- Include Camera -->
-  <xacro:include filename="$(find spooder_description)/urdf/camera.xacro"/>
-  <!-- Include LiDAR -->
+  <!-- Include OAK-D Lite Camera (Gazebo simulation plugin) -->
+  <xacro:include filename="$(find spooder_description)/urdf/gazebo_oakd.plugin.xacro"/>
+  <!-- Include LiDAR (kept for backward compatibility) -->
   <xacro:include filename="$(find spooder_description)/urdf/lidar.xacro"/>
   <!-- Include IMU -->
@@ -43,5 +43,10 @@
     <parent link="base_footprint"/>
     <child link="base_link"/>
-    <origin xyz="0 0 ${tibia_length + 0.05}" rpy="0 0 0"/>
+    <!-- base_link Z above base_footprint. Must be <= FEMUR+TIBIA(0.164) - step_room so
+         the leg can reach the floor at the nominal stance.  Previous value
+         (tibia_length + 0.05 = 0.154) was 19mm too high: default foot
+         (0.12, 0, -0.158) sat 12mm OUTSIDE leg reach, every IK returned (0,0,0),
+         and the body pancakes.  0.135m leaves 18mm margin at (0.085, 0, -0.140). -->
+    <origin xyz="0 0 0.135" rpy="0 0 0"/>
   </joint>
   <!-- Leg Macro -->
@@ -146,6 +151,7 @@
       <gazebo reference="${prefix}_tibia_link">
         <self_collide>false</self_collide>
-        <mu1>1.0</mu1>
-        <mu2>1.0</mu2>
+        <mu1>2.5</mu1>
+        <mu2>2.5</mu2>
+        <min_depth>0.001</min_depth>
         <kp>100000.0</kp>
         <kd>10.0</kd>
@@ -162,6 +168,14 @@
   <xacro:leg prefix="lm" side_sign="1"  x_offset="0.0" y_offset="0.063"  yaw="1.5708"/>
   <xacro:leg prefix="lr" side_sign="1"  x_offset="-0.0835" y_offset="0.063"  yaw="2.3561"/>
-  <!-- Depth Camera -->
-  <xacro:depth_camera parent_link="base_link" origin_xyz="0.095 0 0.15" origin_rpy="0 0 0"/>
+  <!-- OAK-D Lite Depth Camera (replaces generic depth_camera).
+       Mount position: 9.5 cm forward of base_link, 8 cm up. The downward
+       tilt (~20 deg) is set inside the sensor's own <pose> tag so the caller
+       can keep origin_rpy="0 0 0" without double-counting rotations.
+       At 21.5 cm total height (13.5 cm of base_joint + 8 cm mount) and -20 deg
+       pitch, the camera's near clip (0.2 m) hits floor ~0.7 m in front of
+       robot, and the FOV captures the floor up to ~5 m + the horizon. -->
+  <xacro:gazebo_oakd_sensor parent_link="base_link" origin_xyz="0.095 0 0.08" origin_rpy="0 0 0"/>
+  <!-- LiDAR Sensor (kept for backward compatibility) -->
+  <xacro:lidar_sensor parent="base_link"/>
   <!-- ros2_control -->
   <ros2_control name="SpooderSystem" type="system">
